File: main/CE_TestBoard/CE_TestBoard.kicad_pcb (KiCad board)
At the start: 2 copper layers, 145.1 x 56.1 mm, 29 parts, among them Q1 2N2222

Commit message: Repository has been reorganised + new safety changes and minor improvements
Routing:
- net AC: track 225.4 -> 177.5 mm
- net Net-(V2-+): track 103.6 -> 125.2 mm
- net Net-(C2-Pad1): track 54.1 -> 50.8 mm
Other:
- board text added: "v1.0 CE_AMPLIFIER"
Changed lines of the file:
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@@
 			(outputformat 1)
 			(mirror no)
-			(drillshape 1)
+			(drillshape 0)
 			(scaleselection 1)
-			(outputdirectory "")
+			(outputdirectory "pliki wykonawcze wzmacniacz wspolny emiter/")
 		)
 	)
@@
 		)
 	)
+	(gr_text "v1.0 CE_AMPLIFIER"
+		(at 108.25 158.25 0)
+		(layer "F.SilkS")
+		(effects
+			(font
+				(size 1.5 1.5)
+				(thickness 0.3)
+				(bold yes)
+			)
+			(justify left bottom)
+		)
+	)
 	(gr_text "C"
 		(at 164.75 128.5 270)
@@
 	)
 	(segment
-		(start 165.045 115.955)
-		(end 170.25 110.75)
+		(start 170.25 110.75)
+		(end 214.5 110.75)
 		(width 0.8)
 		(layer "F.Cu")
@@
 	)
 	(segment
-		(start 170.25 110.75)
-		(end 179 110.75)
+		(start 233.955 144.295)
+		(end 227.9225 144.295)
 		(width 0.8)
 		(layer "F.Cu")
@@
 	)
 	(segment
-		(start 140.3275 115.955)
-		(end 165.045 115.955)
+		(start 165.045 115.955)
+		(end 170.25 110.75)
 		(width 0.8)
 		(layer "F.Cu")
@@
 	)
 	(segment
-		(start 179 110.75)
-		(end 212.545 144.295)
+		(start 235.5 142.75)
+		(end 233.955 144.295)
 		(width 0.8)
 		(layer "F.Cu")
@@
 	)
 	(segment
-		(start 212.545 144.295)
-		(end 227.9225 144.295)
+		(start 140.3275 115.955)
+		(end 165.045 115.955)
 		(width 0.8)
 		(layer "F.Cu")
@@
 	)
 	(segment
-		(start 211 124.75)
-		(end 213.4575 124.75)
+		(start 214.5 110.75)
+		(end 235.5 131.75)
 		(width 0.8)
 		(layer "F.Cu")
-		(net 6)
+		(net 5)
 	)
 	(segment
-		(start 196.1725 143.715)
-		(end 187.5 152.3875)
+		(start 235.5 131.75)
+		(end 235.5 142.75)
 		(width 0.8)
 		(layer "F.Cu")
-		(net 6)
+		(net 5)
 	)
 	(segment
-		(start 170.75 152.75)
-		(end 187.1375 152.75)
+		(start 213 152)
+		(end 212.5 152.5)
 		(width 0.8)
 		(layer "F.Cu")
@@
 	)
 	(segment
-		(start 210.715 124.465)
-		(end 211 124.75)
+		(start 173.25 150.25)
+		(end 189.6375 150.25)
 		(width 0.8)
 		(layer "F.Cu")
@@
 	)
 	(segment
-		(start 187.5 152.3875)
-		(end 187.5 153.25)
+		(start 211 124.75)
+		(end 213.4575 124.75)
 		(width 0.8)
 		(layer "F.Cu")
@@
 	)
 	(segment
-		(start 232.465 139.215)
-		(end 227.9225 139.215)
+		(start 209.6725 124.465)
+		(end 213 127.7925)
 		(width 0.8)
 		(layer "F.Cu")
@@
 	)
 	(segment
-		(start 103.5775 144.535)
-		(end 106.705 144.535)
+		(start 210.715 124.465)
+		(end 211 124.75)
 		(width 0.8)
 		(layer "F.Cu")
@@
 	)
 	(segment
-		(start 196.1725 143.715)
-		(end 187.1375 152.75)
+		(start 213 127.7925)
+		(end 213 152)
 		(width 0.8)
 		(layer "F.Cu")
@@
 	)
 	(segment
-		(start 170.5775 152.785)
-		(end 170.715 152.785)
+		(start 170.715 152.785)
+		(end 173.25 150.25)
 		(width 0.8)
 		(layer "F.Cu")
@@
 	)
 	(segment
-		(start 232.5 152.75)
-		(end 232.5 139.25)
+		(start 103.5775 144.535)
+		(end 106.705 144.535)
 		(width 0.8)
 		(layer "F.Cu")
@@
 	)
 	(segment
-		(start 232.5 139.25)
-		(end 232.465 139.215)
+		(start 212.5 152.5)
+		(end 191.8875 152.5)
 		(width 0.8)
 		(layer "F.Cu")
@@
 	)
 	(segment
-		(start 187.5 153.25)
-		(end 232 153.25)
+		(start 189.6375 150.25)
+		(end 196.1725 143.715)
 		(width 0.8)
 		(layer "F.Cu")
@@
 	)
 	(segment
-		(start 170.715 152.785)
-		(end 170.75 152.75)
+		(start 170.5775 152.785)
+		(end 170.715 152.785)
 		(width 0.8)
 		(layer "F.Cu")
@@
 	)
 	(segment
-		(start 139.705 148.785)
-		(end 140 149.08)
+		(start 191.8875 152.5)
+		(end 189.6375 150.25)
 		(width 0.8)
 		(layer "F.Cu")
@@
 	)
 	(segment
-		(start 232 153.25)
-		(end 232.5 152.75)
+		(start 139.705 148.785)
+		(end 140 149.08)
 		(width 0.8)
 		(layer "F.Cu")
@@
 	)
 	(segment
-		(start 196.1725 137.965)
-		(end 209.6725 124.465)
-		(width 0.8)
-		(layer "B.Cu")
-		(net 6)
-	)
-	(segment
-		(start 196.1725 143.715)
-		(end 196.1725 137.965)
-		(width 0.8)
-		(layer "B.Cu")
-		(net 6)
-	)
-	(segment
-		(start 186.795 127.5775)
-		(end 198.5 139.2825)
+		(start 209.6725 135.295)
+		(end 196.1725 148.795)
 		(width 0.8)
 		(layer "F.Cu")
@@
 	)
 	(segment
-		(start 198.5 139.2825)
-		(end 198.5 146.4675)
+		(start 209.6725 129.545)
+		(end 209.6725 135.295)
 		(width 0.8)
 		(layer "F.Cu")
@@
 	)
 	(segment
-		(start 198.5 146.4675)
-		(end 196.1725 148.795)
+		(start 186.795 127.5775)
+		(end 207.705 127.5775)
 		(width 0.8)
 		(layer "F.Cu")
@@
 	)
 	(segment
-		(start 197.7735 147.194)
-		(end 196.1725 148.795)
+		(start 207.705 127.5775)
+		(end 209.6725 129.545)
 		(width 0.8)
-		(layer "B.Cu")
+		(layer "F.Cu")
 		(net 7)
 	)
 	(segment
-		(start 209.6725 135.295)
+		(start 197.7735 147.194)
 		(end 196.1725 148.795)
 		(width 0.8)
 		(layer "B.Cu")
-		(net 7)
-	)
-	(segment
-		(start 209.6725 129.545)
-		(end 209.6725 135.295)
-		(width 0.8)
-		(layer "B.Cu")
