File: main/CE_TestBoard/CE_TestBoard.kicad_pcb (KiCad board)
At the start: 2 copper layers, 145.1 x 56.1 mm, 29 parts, among them Q1 2N2222

Commit message: Minor fixes
Parts:
- moved G*** 95.5 mm to (203.0, 114.8), turned to 180 degrees
- moved D1 82.5 mm to (196.2, 110.8), turned to 0 degrees
Connections:
- C1 pad 2: Net-(D1-K) -> Net-(V1-+)
- D1 pad 1: Net-(D1-K) -> Net-(D2-K)
- D1 pad 2: Net-(D1-A) -> Net-(D2-A)
- R1 pad 1: Net-(V2-+) -> Net-(D2-K)
- RC1 pad 1: Net-(V2-+) -> Net-(D2-K)
- V1 pad 1: Net-(D1-A) -> Net-(V1-+)
- V2 pad 1: Net-(V2-+) -> Net-(D2-A)
Routing:
- net Net-(V2-+): track 103.6 -> 0.00 mm
- net Net-(D2-K): track 0.00 -> 58.0 mm
- net Net-(D2-A): track 0.00 -> 56.8 mm
- net AC: track 225.4 -> 177.5 mm
- net Net-(V1-+): track 0.00 -> 30.8 mm
- net Net-(D1-A): track 15.3 -> 0.00 mm
- net Net-(D1-K): track 5.64 -> 0.00 mm
- net Net-(C2-Pad1): track 54.1 -> 50.8 mm
Other:
- board text added: "v1.0 CE_AMPLIFIER"
