File: main/OpAmp_TestBoard/OpAmp_TestBoard.kicad_pcb (KiCad board)
At the start: 2 copper layers, 145.1 x 56.1 mm, 28 parts, among them U1 LM358

Commit message: Repository has been reorganised + new safety changes and minor improvements
Parts:
- added G***: LOGO, kicad moje pliki:Triangle_wave_logo, F.Cu at (211.0, 74.2)
- added G***: LOGO, kicad moje pliki:Square_wave_logo, F.Cu at (174.2, 51.0)
Connections:
- net Net-(D1-K) renamed VCC
- C1 pad 1: GND -> GNDA
- C1 pad 2: Net-(U1-V-) -> GND
- C2 pad 2: GND -> GNDA
- R4 pad 2: GND -> GNDA
- R5 pad 1: GND -> GNDA
- R5 pad 2: Net-(U1-V-) -> GND
- R6 pad 2: GND -> GNDA
- R7 pad 2: GND -> GNDA
- U1 pad 2: GND -> GNDA
- U1 pad 4: Net-(U1-V-) -> GND
- U1 pad 5: GND -> GNDA
- V1 pad 2: Net-(U1-V-) -> GND
Routing:
- net GNDA: track 0.00 -> 165.1 mm
- net Net-(U1-V-): track 85.4 -> 0.00 mm
- net GND: track 165.1 -> 85.4 mm
Other:
- board text added: "v1.0 GEN_TRIANGLE_SQUARE"
