File: main/OpAmp_TestBoard/OpAmp_TestBoard.kicad_sch (KiCad schematic)
At the start: 13 parts, among them U1 LM358

Commit message: Repository has been reorganised + new safety changes and minor improvements
Connections:
- net GND: now also C1.2, R5.2, U1.4 (V-), V1.2 (-); no longer C1.1, C2.2, R4.2, R5.1, R6.2, R7.2, U1.2 (A-), U1.5 (B+)
- net VCC: now reaches C2.1, D1.1 (K), R4.1, U1.8 (V+)
- new net GNDA: C1.1, C2.2, R4.2, R5.1, R6.2, R7.2, U1.2 (A-), U1.5 (B+)
Other:
- moved on the sheet: C1, C2, D1, R3, V1
